File: SpotWelder.kicad_sch (KiCad schematic)
At the start: 12 parts, among them J1 Conn_01x01_Pin, J2 Conn_01x01_Pin, SW1 SW_WELD, SW2 SW_UP, SW3 SW_DOWN, SW4 SW_WELD_WHILE_HELD, U1 Beetle_DFR0282, U3 LM7805_TO220

Commit message: Add files via upload
Other:
- note added: "BLK"
- note added: "BLU"
- note added: "BRN"
- note added: "GRN"
- note added: "Note 1: Pressing both Up and Down together will enter into setup mode allowing the default time period for Up and Down button presses to be changed. Potentially you will also be able to set a 'pre weld' period to initially heat the metal before the final weld. The Weld button selects the mode while in setup mode. Pressing the UntimedWeld button while in setup mode will return you to normal operat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"
- note added: "RED"
- note added: "YEL"
- note removed: "Note 1: Pressing both Up and Down together will enter into setup mode allowing the default time period for Up and Down button presses to be changed. Potentially you will also be able to set a 'pre weld' period to initially heat the metal before the final weld. The Weld button selects the mode while in setup mode. Pressing Up and Down buttons a second time return you to normal operation"
Changed lines of the file:
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@@
 	(title_block
 		(title "Spot Welder")
-		(date "24 Feb 2026")
-		(rev "V1")
+		(date "15 Mar 2026")
+		(rev "V1.1")
 		(comment 4 "Greg George")
+	)
+	(text "GRN"
+		(exclude_from_sim no)
+		(at 185.166 130.048 0)
+		(effects
+			(font
+				(size 1.27 1.27)
+			)
+		)
+	)
+	(text "RED"
+		(exclude_from_sim no)
+		(at 144.018 94.234 0)
+		(effects
+			(font
+				(size 1.27 1.27)
+			)
+		)
+	)
+	(text "YEL"
+		(exclude_from_sim no)
+		(at 169.926 130.302 0)
+		(effects
+			(font
+				(size 1.27 1.27)
+			)
+		)
 	)
 	(text "240VAC"
@@
 		)
 	)
-	(text "Note 1: \n\nPressing both Up and Down together will enter into\nsetup mode allowing the default time period for Up\nand Down button presses to be changed.  Potentially\nyou will also be able to set a 'pre weld' period to \ninitially heat the metal before the final weld.\n\nThe Weld button selects the mode while in setup mode.\n\nPressing Up and Down buttons a second time return you\nto normal operation"
+	(text "Note 1: \n\nPressing both Up and Down together will enter into\nsetup mode allowing the default time period for Up\nand Down button presses to be changed.  Potentially\nyou will also be able to set a 'pre weld' period to \ninitially heat the metal before the final weld.\n\nThe Weld button selects the mode while in setup mode.\n\nPressing the UntimedWeld button while in setup mode\nwill return you to normal operation.\n\nThe maximum UnitmedWeld duration is 10 seconds."
 		(exclude_from_sim no)
 		(at 113.284 178.816 0)
@@
 		(exclude_from_sim no)
 		(at 173.99 118.872 0)
+		(effects
+			(font
+				(size 1.27 1.27)
+			)
+		)
+	)
+	(text "RED"
+		(exclude_from_sim no)
+		(at 129.794 130.048 0)
+		(effects
+			(font
+				(size 1.27 1.27)
+			)
+		)
+	)
+	(text "BLK"
+		(exclude_from_sim no)
+		(at 192.024 130.302 0)
+		(effects
+			(font
+				(size 1.27 1.27)
+			)
+		)
+	)
+	(text "BLK"
+		(exclude_from_sim no)
+		(at 138.43 131.318 0)
+		(effects
+			(font
+				(size 1.27 1.27)
+			)
+		)
+	)
+	(text "BLK"
+		(exclude_from_sim no)
+		(at 110.49 127.508 0)
+		(effects
+			(font
+				(size 1.27 1.27)
+			)
+		)
+	)
+	(text "BLU"
+		(exclude_from_sim no)
+		(at 150.622 129.794 0)
 		(effects
 			(font
@@
 		)
 	)
+	(text "BLK"
+		(exclude_from_sim no)
+		(at 159.004 131.318 0)
+		(effects
+			(font
+				(size 1.27 1.27)
+			)
+		)
+	)
+	(text "BLK"
+		(exclude_from_sim no)
+		(at 177.546 132.588 0)
+		(effects
+			(font
+				(size 1.27 1.27)
+			)
+		)
+	)
 	(text "240VAC Mains Power"
 		(exclude_from_sim no)
@@
 		(effects
 			(font
+				(size 1.27 1.27)
+			)
+		)
+	)
+	(text "BRN"
+		(exclude_from_sim no)
+		(at 141.732 102.87 0)
+		(effects
+			(font
